File: 7SegV10.kicad_pcb (KiCad board)
At the start: 2 copper layers, 100 x 150 mm, 74 parts, among them IC1 ATMEGA328-A, P1 GPIO1 STM32, P10 Power In, P11 USB STM32, P2 GPIO2 STM32, P3 RS232 STM32, P4 SWD, P5 GPIO1 AVR, P6 RS232 AVR, P7 ISP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

Commit message: new version
Connections:
- U3 pad 5: VCC -> +5V
Routing:
- net +5V: track 17.4 -> 23.5 mm
- net VCC: track 6.03 -> 0.00 mm
- net RESET_AVR: track 51.0 -> 52.1 mm
- net Net-(IC1-Pad17): track 15.0 -> 16.0 mm
- net GND: track 165.1 -> 164.4 mm
Other:
- board text added: "Back"
- board text added: "Front"
